File: hardware/kicad/ATO_Controller.kicad_sch (KiCad schematic)
At the start: 26 parts, among them J1 USB_C_24pin, J2 USB_A_Pump_Output, J3 LOW_SENSOR_JST-XH, J4 HIGH_SENSOR_JST-XH, J5 EXPANSION_JST-XH, J6 RESERVOIR_JST-XH, Q1 2N2222, SW1 SPST_5A, U1_SOCKET XIAO_ESP32S3_SOCKET

Commit message: Regenerate KiCad schematic with improved layout and complete connections
Parts:
- removed C2 (x2): 100nF, symbol Device:C
- removed U1_SOCKET: XIAO_ESP32S3_SOCKET, symbol Connector:Conn_01x20_Female
- added C2 (x2): 100nF, symbol Device:C
- added U1: XIAO_ESP32S3_SOCKET, symbol Connector:Conn_01x16_Female
- C1: value 470µF/10V -> 470uF_10V
- F1: value MF-R150 -> MF-R150_1.5A
- J2: value USB_A_Pump_Output -> USB_A_PUMP
- LED1: value LED_GREEN_PWR -> LED_GREEN
- LED2: value LED_BLUE_PUMP -> LED_BLUE
- LED3: value LED_RED_ERR -> LED_RED
- LED4: value LED_AMBER_RELAY -> LED_AMBER
- R1: value 10kΩ -> 10k
- R2, R3, R4, R5: value 330Ω -> 330
Other:
- note added: "MICROCONTROLLER"
- note added: "POWER INPUT"
- note added: "RELAY CONTROL"
- note added: "SENSORS"
- note removed: "MCU SECTION"
- note removed: "POWER INPUT SECTION"
- note removed: "PUMP OUTPUT SECTION"
- note removed: "RELAY CONTROL SECTION"
- note removed: "SENSOR CONNECTORS"
- company: DIY Project -> DIY Aquarium Project
- title: Aquarium ATO Controller -> Aquarium ATO Controller PCBA
